File: kicad/7Backpack.kicad_pcb (KiCad board)
At the start: 2 copper layers, 14 x 83.2 mm, 14 parts, among them J1 Conn_01x06, J2 Conn_01x06, U1 TPIC6C596PWR, U2 15101BS-30101BS

Commit message: Autorouted
Parts:
- moved C1 0.51 mm to (100.3, 100.5), turned to 90 degrees
- moved R1 0.41 mm to (100.3, 104.8)
Routing:
- net Net-(R6-Pad1): track 0.00 -> 42.7 mm
- net Net-(R4-Pad1): track 0.00 -> 27.8 mm
- net Net-(R5-Pad1): track 0.00 -> 26.0 mm
- net Net-(J1-Pad3): track 0.00 -> 25.6 mm
- net +5V: track 8.89 -> 33.5 mm
- net Net-(J1-Pad4): track 0.00 -> 19.8 mm, vias 0 -> 1
- net Net-(J1-Pad2): track 0.00 -> 19.3 mm
- net Net-(J2-Pad3): track 0.00 -> 14.7 mm
- net Net-(R3-Pad1): track 0.00 -> 11.7 mm, vias 0 -> 2
- net Net-(R8-Pad1): track 0.00 -> 10.3 mm, vias 0 -> 2
- net GND: track 0.00 -> 10.2 mm, vias 0 -> 2
- net Net-(R7-Pad1): track 0.00 -> 7.78 mm, vias 0 -> 2
- net Net-(R9-Pad1): track 0.00 -> 6.98 mm
- net Net-(R2-Pad1): track 0.19 -> 6.68 mm
- net Net-(R1-Pad1): track 0.00 -> 3.89 mm

Commit message: Finalized routing
Parts:
- moved R1 0.90 mm to (101.0, 104.1)
- moved C1 0.64 mm to (101.0, 100.5)
Routing:
- net GND: track 10.2 -> 5.32 mm, vias 2 -> 3
- net Net-(R1-Pad1): track 3.89 -> 2.99 mm
- net +5V: track 33.5 -> 32.6 mm
- net Net-(R8-Pad1): track 10.3 -> 9.82 mm, vias 2 -> 0
- net Net-(R9-Pad1): track 6.98 -> 7.08 mm, vias 0 -> 2
- net Net-(R7-Pad1): track 7.78 -> 7.74 mm, vias 2 -> 0
- added copper zone on B.Cu, net GND
Other:
- board text added: "(cc) BY-NC-SA - 2024 www.agius-industries.eu"
- board text added: "+5V"
- board text added: "7Backpack v1.0"
- board text added: "CLOCK"
- board text added: "GND"
- board text added: "IN"
- board text added: "LATCH"
- board text added: "OUT"
- board text added: "VCC"
