File: kicad/7Backpack.kicad_sch (KiCad schematic)
At the start: 14 parts, among them J1 Conn_01x06, J2 Conn_01x06, U1 TPIC6C596PWR, U2 15101BS-30101BS

Commit message: AddedGerber files
Parts:
- C1: LCSC (none) -> C14663
- R1: LCSC (none) -> C25804
- R2, R3, R4, R5, R6, R7, R8: LCSC (none) -> C22810
- R9: value 30Ω ? -> 2kΩ; LCSC (none) -> C22975
- U1: LCSC (none) -> C3304552; Package TSSOP-16 Texas Instruments -> (none)
Changed lines of the file:
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@@
   )
   (symbol (lib_id "Device:R") (at 163.83 71.755 90) (unit 1)
-    (in_bom yes) (on_board yes) (fields_autoplaced)
-    (property "Reference" "R2" (id 0) (at 163.83 66.04 90))
-    (property "Value" "15Ω" (id 1) (at 163.83 68.58 90))
+    (in_bom yes) (on_board yes)
+    (property "Reference" "R2" (id 0) (at 162.56 69.85 90))
+    (property "Value" "15Ω" (id 1) (at 167.64 69.85 90))
     (property "Footprint" "Resistor_SMD:R_0603_1608Metric" (id 2) (at 163.83 73.533 90)
       (effects (font (size 1.27 1.27)) hide)
     )
     (property "Datasheet" "~" (id 3) (at 163.83 71.755 0)
+      (effects (font (size 1.27 1.27)) hide)
+    )
+    (property "LCSC" "C22810" (id 4) (at 163.83 71.755 90)
       (effects (font (size 1.27 1.27)) hide)
     )
@@
       (effects (font (size 1.27 1.27)) hide)
     )
+    (property "LCSC" "C14663" (id 4) (at 66.04 78.105 0)
+      (effects (font (size 1.27 1.27)) hide)
+    )
     (pin "1")
     (pin "2")
@@
   )
   (symbol (lib_id "Device:R") (at 163.83 97.155 90) (unit 1)
-    (in_bom yes) (on_board yes) (fields_autoplaced)
-    (property "Reference" "R7" (id 0) (at 163.83 91.44 90))
-    (property "Value" "15Ω" (id 1) (at 163.83 93.98 90))
+    (in_bom yes) (on_board yes)
+    (property "Reference" "R7" (id 0) (at 162.56 95.25 90))
+    (property "Value" "15Ω" (id 1) (at 167.64 95.25 90))
     (property "Footprint" "Resistor_SMD:R_0603_1608Metric" (id 2) (at 163.83 98.933 90)
       (effects (font (size 1.27 1.27)) hide)
     )
     (property "Datasheet" "~" (id 3) (at 163.83 97.155 0)
+      (effects (font (size 1.27 1.27)) hide)
+    )
+    (property "LCSC" "C22810" (id 4) (at 163.83 97.155 0)
       (effects (font (size 1.27 1.27)) hide)
     )
@@
       (effects (font (size 1.27 1.27)) hide)
     )
+    (property "LCSC" "C25804" (id 4) (at 78.74 78.105 0)
+      (effects (font (size 1.27 1.27)) hide)
+    )
     (pin "1")
     (pin "2")
@@
   )
   (symbol (lib_id "Device:R") (at 163.83 92.075 90) (unit 1)
-    (in_bom yes) (on_board yes) (fields_autoplaced)
-    (property "Reference" "R6" (id 0) (at 163.83 86.36 90))
-    (property "Value" "15Ω" (id 1) (at 163.83 88.9 90))
+    (in_bom yes) (on_board yes)
+    (property "Reference" "R6" (id 0) (at 162.56 90.17 90))
+    (property "Value" "15Ω" (id 1) (at 167.64 90.17 90))
     (property "Footprint" "Resistor_SMD:R_0603_1608Metric" (id 2) (at 163.83 93.853 90)
       (effects (font (size 1.27 1.27)) hide)
     )
     (property "Datasheet" "~" (id 3) (at 163.83 92.075 0)
+      (effects (font (size 1.27 1.27)) hide)
+    )
+    (property "LCSC" "C22810" (id 4) (at 163.83 92.075 0)
       (effects (font (size 1.27 1.27)) hide)
     )
@@
   )
   (symbol (lib_id "Device:R") (at 163.83 107.315 90) (unit 1)
-    (in_bom yes) (on_board yes) (fields_autoplaced)
-    (property "Reference" "R9" (id 0) (at 163.83 101.6 90))
-    (property "Value" "30Ω ?" (id 1) (at 163.83 104.14 90))
+    (in_bom yes) (on_board yes)
+    (property "Reference" "R9" (id 0) (at 162.56 105.41 90))
+    (property "Value" "2kΩ" (id 1) (at 167.64 105.41 90))
     (property "Footprint" "Resistor_SMD:R_0603_1608Metric" (id 2) (at 163.83 109.093 90)
       (effects (font (size 1.27 1.27)) hide)
@@
       (effects (font (size 1.27 1.27)) hide)
     )
+    (property "LCSC" "C22975" (id 4) (at 163.83 107.315 0)
+      (effects (font (size 1.27 1.27)) hide)
+    )
     (pin "1")
     (pin "2")
   )
   (symbol (lib_id "Device:R") (at 163.83 102.235 90) (unit 1)
-    (in_bom yes) (on_board yes) (fields_autoplaced)
-    (property "Reference" "R8" (id 0) (at 163.83 96.52 90))
-    (property "Value" "15Ω" (id 1) (at 163.83 99.06 90))
+    (in_bom yes) (on_board yes)
+    (property "Reference" "R8" (id 0) (at 162.56 100.33 90))
+    (property "Value" "15Ω" (id 1) (at 167.64 100.33 90))
     (property "Footprint" "Resistor_SMD:R_0603_1608Metric" (id 2) (at 163.83 104.013 90)
       (effects (font (size 1.27 1.27)) hide)
     )
     (property "Datasheet" "~" (id 3) (at 163.83 102.235 0)
+      (effects (font (size 1.27 1.27)) hide)
+    )
+    (property "LCSC" "C22810" (id 4) (at 163.83 102.235 0)
       (effects (font (size 1.27 1.27)) hide)
     )
@@
       (effects (font (size 1.27 1.27)) hide)
     )
-    (property "Description" "\nAutomotive 8-bit shift register\n" (id 5) (at 116.205 84.455 0)
-      (effects (font (size 1.27 1.27)) (justify bottom) hide)
-    )
     (property "PACKAGE" "TSSOP-16" (id 6) (at 116.205 84.455 0)
       (effects (font (size 1.27 1.27)) (justify bottom) hide)
@@
       (effects (font (size 1.27 1.27)) (justify bottom) hide)
     )
-    (property "Package" "TSSOP-16 Texas Instruments" (id 9) (at 116.205 84.455 0)
-      (effects (font (size 1.27 1.27)) (justify bottom) hide)
+    (property "LCSC" "C3304552" (id 6) (at 116.205 84.455 0)
+      (effects (font (size 1.27 1.27)) hide)
     )
     (pin "1")
@@
   )
   (symbol (lib_id "Device:R") (at 163.83 81.915 90) (unit 1)
-    (in_bom yes) (on_board yes) (fields_autoplaced)
-    (property "Reference" "R4" (id 0) (at 163.83 76.2 90))
-    (property "Value" "15Ω" (id 1) (at 163.83 78.74 90))
+    (in_bom yes) (on_board yes)
+    (property "Reference" "R4" (id 0) (at 162.56 80.01 90))
+    (property "Value" "15Ω" (id 1) (at 167.64 80.01 90))
     (property "Footprint" "Resistor_SMD:R_0603_1608Metric" (id 2) (at 163.83 83.693 90)
       (effects (font (size 1.27 1.27)) hide)
     )
     (property "Datasheet" "~" (id 3) (at 163.83 81.915 0)
+      (effects (font (size 1.27 1.27)) hide)
+    )
+    (property "LCSC" "C22810" (id 4) (at 163.83 81.915 0)
       (effects (font (size 1.27 1.27)) hide)
     )
@@
   )
   (symbol (lib_id "Device:R") (at 163.83 76.835 90) (unit 1)
-    (in_bom yes) (on_board yes) (fields_autoplaced)
-    (property "Reference" "R3" (id 0) (at 163.83 71.12 90))
-    (property "Value" "15Ω" (id 1) (at 163.83 73.66 90))
+    (in_bom yes) (on_board yes)
+    (property "Reference" "R3" (id 0) (at 162.56 74.93 90))
+    (property "Value" "15Ω" (id 1) (at 167.64 74.93 90))
     (property "Footprint" "Resistor_SMD:R_0603_1608Metric" (id 2) (at 163.83 78.613 90)
       (effects (font (size 1.27 1.27)) hide)
@@
       (effects (font (size 1.27 1.27)) hide)
     )
+    (property "LCSC" "C22810" (id 4) (at 163.83 76.835 0)
+      (effects (font (size 1.27 1.27)) hide)
+    )
     (pin "1")
     (pin "2")
   )
   (symbol (lib_id "Device:R") (at 163.83 86.995 90) (unit 1)
-    (in_bom yes) (on_board yes) (fields_autoplaced)
-    (property "Reference" "R5" (id 0) (at 163.83 81.28 90))
-    (property "Value" "15Ω" (id 1) (at 163.83 83.82 90))
+    (in_bom yes) (on_board yes)
+    (property "Reference" "R5" (id 0) (at 162.56 85.09 90))
+    (property "Value" "15Ω" (id 1) (at 167.64 85.09 90))
     (property "Footprint" "Resistor_SMD:R_0603_1608Metric" (id 2) (at 163.83 88.773 90)
       (effects (font (size 1.27 1.27)) hide)
     )
     (property "Datasheet" "~" (id 3) (at 163.83 86.995 0)
+      (effects (font (size 1.27 1.27)) hide)
+    )
+    (property "LCSC" "C22810" (id 4) (at 163.83 86.995 0)
       (effects (font (size 1.27 1.27)) hide)
     )
@@
     )
     (path "/bb886b81-57b9-4350-992a-f0311e5b361d"
-      (reference "R9") (unit 1) (value "30Ω ?") (footprint "Resistor_SMD:R_0603_1608Metric")
+      (reference "R9") (unit 1) (value "2kΩ") (footprint "Resistor_SMD:R_0603_1608Metric")
     )
     (path "/cf963df9-70b8-447a-b4bc-d4607209d73a"

Commit message: Switched to SOP-16
Parts:
- R1: value 10kΩ -> 10k
- R2, R3, R4, R5, R6, R7, R8: value 15Ω -> 15
- R9: value 2kΩ -> 2k
- U1: value TPIC6C596PWR -> TPIC6C596DC; footprint TPIC6C596PWR:SOP65P640X120-16N -> TPIC6C596DR:SOIC127P600X175-16N; LCSC C3304552 -> C2872253; MPN TPIC6C596PWR -> (none); PACKAGE TSSOP-16 -> SOIC-16
Changed lines of the file:
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@@
     (in_bom yes) (on_board yes)
     (property "Reference" "R2" (id 0) (at 162.56 69.85 90))
-    (property "Value" "15Ω" (id 1) (at 167.64 69.85 90))
+    (property "Value" "15" (id 1) (at 167.64 69.85 90))
     (property "Footprint" "Resistor_SMD:R_0603_1608Metric" (id 2) (at 163.83 73.533 90)
       (effects (font (size 1.27 1.27)) hide)
@@
     (in_bom yes) (on_board yes)
     (property "Reference" "R7" (id 0) (at 162.56 95.25 90))
-    (property "Value" "15Ω" (id 1) (at 167.64 95.25 90))
+    (property "Value" "15" (id 1) (at 167.64 95.25 90))
     (property "Footprint" "Resistor_SMD:R_0603_1608Metric" (id 2) (at 163.83 98.933 90)
       (effects (font (size 1.27 1.27)) hide)
@@
       (effects (font (size 1.27 1.27)) (justify right))
     )
-    (property "Value" "10kΩ" (id 1) (at 81.28 79.3749 0)
+    (property "Value" "10k" (id 1) (at 81.28 79.3749 0)
       (effects (font (size 1.27 1.27)) (justify right))
     )
@@
     (in_bom yes) (on_board yes)
     (property "Reference" "R6" (id 0) (at 162.56 90.17 90))
-    (property "Value" "15Ω" (id 1) (at 167.64 90.17 90))
+    (property "Value" "15" (id 1) (at 167.64 90.17 90))
     (property "Footprint" "Resistor_SMD:R_0603_1608Metric" (id 2) (at 163.83 93.853 90)
       (effects (font (size 1.27 1.27)) hide)
@@
     (in_bom yes) (on_board yes)
     (property "Reference" "R9" (id 0) (at 162.56 105.41 90))
-    (property "Value" "2kΩ" (id 1) (at 167.64 105.41 90))
+    (property "Value" "2k" (id 1) (at 167.64 105.41 90))
     (property "Footprint" "Resistor_SMD:R_0603_1608Metric" (id 2) (at 163.83 109.093 90)
       (effects (font (size 1.27 1.27)) hide)
@@
     (in_bom yes) (on_board yes)
     (property "Reference" "R8" (id 0) (at 162.56 100.33 90))
-    (property "Value" "15Ω" (id 1) (at 167.64 100.33 90))
+    (property "Value" "15" (id 1) (at 167.64 100.33 90))
     (property "Footprint" "Resistor_SMD:R_0603_1608Metric" (id 2) (at 163.83 104.013 90)
       (effects (font (size 1.27 1.27)) hide)
@@
     (in_bom yes) (on_board yes) (fields_autoplaced)
     (property "Reference" "U1" (id 0) (at 116.205 66.675 0))
-    (property "Value" "TPIC6C596PWR" (id 1) (at 116.205 69.215 0))
-    (property "Footprint" "TPIC6C596PWR:SOP65P640X120-16N" (id 2) (at 116.205 84.455 0)
+    (property "Value" "TPIC6C596DC" (id 1) (at 116.205 69.215 0))
+    (property "Footprint" "TPIC6C596DR:SOIC127P600X175-16N" (id 2) (at 116.205 84.455 0)
       (effects (font (size 1.27 1.27)) (justify bottom) hide)
     )
@@
       (effects (font (size 1.27 1.27)) hide)
     )
-    (property "PACKAGE" "TSSOP-16" (id 6) (at 116.205 84.455 0)
+    (property "PACKAGE" "SOIC-16" (id 6) (at 116.205 84.455 0)
       (effects (font (size 1.27 1.27)) (justify bottom) hide)
     )
-    (property "MPN" "TPIC6C596PWR" (id 7) (at 116.205 84.455 0)
-      (effects (font (size 1.27 1.27)) (justify bottom) hide)
-    )
-    (property "LCSC" "C3304552" (id 6) (at 116.205 84.455 0)
+    (property "LCSC" "C2872253" (id 7) (at 116.205 84.455 0)
       (effects (font (size 1.27 1.27)) hide)
     )
@@
     (in_bom yes) (on_board yes)
     (property "Reference" "R4" (id 0) (at 162.56 80.01 90))
-    (property "Value" "15Ω" (id 1) (at 167.64 80.01 90))
+    (property "Value" "15" (id 1) (at 167.64 80.01 90))
     (property "Footprint" "Resistor_SMD:R_0603_1608Metric" (id 2) (at 163.83 83.693 90)
       (effects (font (size 1.27 1.27)) hide)
@@
     (in_bom yes) (on_board yes)
     (property "Reference" "R3" (id 0) (at 162.56 74.93 90))
-    (property "Value" "15Ω" (id 1) (at 167.64 74.93 90))
+    (property "Value" "15" (id 1) (at 167.64 74.93 90))
     (property "Footprint" "Resistor_SMD:R_0603_1608Metric" (id 2) (at 163.83 78.613 90)
       (effects (font (size 1.27 1.27)) hide)
@@
     (in_bom yes) (on_board yes)
     (property "Reference" "R5" (id 0) (at 162.56 85.09 90))
-    (property "Value" "15Ω" (id 1) (at 167.64 85.09 90))
+    (property "Value" "15" (id 1) (at 167.64 85.09 90))
     (property "Footprint" "Resistor_SMD:R_0603_1608Metric" (id 2) (at 163.83 88.773 90)
       (effects (font (size 1.27 1.27)) hide)
@@
     )
     (path "/867d40ef-7c10-4dba-bd59-2d78cf8e8b70"
-      (reference "R1") (unit 1) (value "10kΩ") (footprint "Resistor_SMD:R_0603_1608Metric")
+      (reference "R1") (unit 1) (value "10k") (footprint "Resistor_SMD:R_0603_1608Metric")
     )
     (path "/208fd5fc-c0c1-4790-9531-2e9af2ccc503"
-      (reference "R2") (unit 1) (value "15Ω") (footprint "Resistor_SMD:R_0603_1608Metric")
+      (reference "R2") (unit 1) (value "15") (footprint "Resistor_SMD:R_0603_1608Metric")
     )
     (path "/fc831169-3f51-47ae-b367-8b992f27cb69"
-      (reference "R3") (unit 1) (value "15Ω") (footprint "Resistor_SMD:R_0603_1608Metric")
+      (reference "R3") (unit 1) (value "15") (footprint "Resistor_SMD:R_0603_1608Metric")
     )
     (path "/ee992d96-582c-47b5-b9cc-730301fd84f6"
-      (reference "R4") (unit 1) (value "15Ω") (footprint "Resistor_SMD:R_0603_1608Metric")
+      (reference "R4") (unit 1) (value "15") (footprint "Resistor_SMD:R_0603_1608Metric")
     )
     (path "/fe8fbdf9-277a-42b8-bf31-c21df22d6ccb"
-      (reference "R5") (unit 1) (value "15Ω") (footprint "Resistor_SMD:R_0603_1608Metric")
+      (reference "R5") (unit 1) (value "15") (footprint "Resistor_SMD:R_0603_1608Metric")
     )
     (path "/a558b1b2-4ec8-4880-8e4b-82c95cf6e997"
-      (reference "R6") (unit 1) (value "15Ω") (footprint "Resistor_SMD:R_0603_1608Metric")
+      (reference "R6") (unit 1) (value "15") (footprint "Resistor_SMD:R_0603_1608Metric")
     )
     (path "/763e4dde-457a-40c1-adc0-2cf92812ab35"
-      (reference "R7") (unit 1) (value "15Ω") (footprint "Resistor_SMD:R_0603_1608Metric")
+      (reference "R7") (unit 1) (value "15") (footprint "Resistor_SMD:R_0603_1608Metric")
     )
     (path "/cefd95e4-1d86-4a10-a24a-f3abbf5db5e4"
-      (reference "R8") (unit 1) (value "15Ω") (footprint "Resistor_SMD:R_0603_1608Metric")
+      (reference "R8") (unit 1) (value "15") (footprint "Resistor_SMD:R_0603_1608Metric")
     )
     (path "/bb886b81-57b9-4350-992a-f0311e5b361d"
-      (reference "R9") (unit 1) (value "2kΩ") (footprint "Resistor_SMD:R_0603_1608Metric")
+      (reference "R9") (unit 1) (value "2k") (footprint "Resistor_SMD:R_0603_1608Metric")
     )
     (path "/cf963df9-70b8-447a-b4bc-d4607209d73a"
-      (reference "U1") (unit 1) (value "TPIC6C596PWR") (footprint "TPIC6C596PWR:SOP65P640X120-16N")
+      (reference "U1") (unit 1) (value "TPIC6C596DC") (footprint "TPIC6C596DR:SOIC127P600X175-16N")
     )
     (path "/effd2c1c-4501-4ff7-bfcb-218d17a34103"
